File: schematics/retrofit/MAHO_Inputs.kicad_sch (KiCad schematic)
At the start: 3 parts, among them U401 7i97-TB5-OUTPUTS-A, U402 7i97-TB5-OUTPUTS-B

Commit message: schematics
Other:
- moved on the sheet: U401, U402
