File: schematics/retrofit/MAHO_Outputs.kicad_sch (KiCad schematic)
At the start: 8 parts, among them J501 LIMIT_X, J502 LIMIT_Y, J503 LIMIT_Z, U501 7i97-TB4-Inputs-A, U502 7i97-TB4-Inputs-B, U503 7i97-TB5-Inputs-C, U504 7i97-TB5-Inputs-D

Commit message: draft
Connections:
- no-connect marks 6 -> 4
Changed lines of the file:
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@@
 (kicad_sch (version 20230121) (generator eeschema)
   (paper "A4")
-  (no_connect (at 82.55 135.89))
   (no_connect (at 82.55 115.57))
   (no_connect (at 82.55 118.11))
   (no_connect (at 82.55 123.19))
   (no_connect (at 82.55 120.65))
-  (no_connect (at 82.55 133.35))
   (wire (pts (xy 187.96 73.66) (xy 201.93 73.66))
     (stroke (width 0) (type default))
