File: schematics/retrofit/PWR.kicad_sch (KiCad schematic)
At the start: 4 parts, among them J601 24V PWR, U601 7i97-TB4-5V

Commit message: schematics
Other:
- moved on the sheet: ESTOP?, J601, PWR_SWITCH?, U601

Commit message: draft
Parts:
- added J602: 12V PWR, symbol Connector_Generic:Conn_01x02
- added J603: 5V PWR, symbol Connector_Generic:Conn_01x02
Connections:
- net GND: now also J602.2 (Pin_2), J603.2 (Pin_2)
- new net 12V: J602.1 (Pin_1)
- new net 5V: J603.1 (Pin_1)
Changed lines of the file:
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@@
+    (stroke (width 0) (type default))
+  )
+  (wire (pts (xy 46.99 83.82) (xy 55.88 83.82))
     (stroke (width 0) (type default))
   )
@@
     (stroke (width 0) (type default))
   )
+  (wire (pts (xy 46.99 95.25) (xy 55.88 95.25))
+    (stroke (width 0) (type default))
+  )
   (wire (pts (xy 142.24 93.98) (xy 152.4 93.98))
     (stroke (width 0) (type default))
@@
     )
   )
+  (global_label "12V" (shape input) (at 55.88 83.82 0) (fields_autoplaced)
+    (effects (font (size 1.27 1.27)) (justify left))
+    (property "Intersheetrefs" "${INTERSHEET_REFS}" (at 62.2934 83.82 0)
+      (effects (font (size 1.27 1.27)) (justify left) hide)
+    )
+  )
   (global_label "204" (shape input) (at 58.42 30.48 0) (fields_autoplaced)
     (effects (font (size 1.27 1.27)) (justify left))
@@
     (effects (font (size 1.27 1.27)) (justify left))
     (property "Intersheetrefs" "${INTERSHEET_REFS}" (at 158.9343 83.82 0)
+      (effects (font (size 1.27 1.27)) (justify left) hide)
+    )
+  )
+  (global_label "5V" (shape input) (at 55.88 95.25 0) (fields_autoplaced)
+    (effects (font (size 1.27 1.27)) (justify left))
+    (property "Intersheetrefs" "${INTERSHEET_REFS}" (at 61.0839 95.25 0)
       (effects (font (size 1.27 1.27)) (justify left) hide)
     )
@@
     )
   )
+  (symbol (lib_id "Connector_Generic:Conn_01x02") (at 41.91 83.82 0) (mirror y) (unit 1)
+    (in_bom yes) (on_board yes) (dnp no)
+    (property "Reference" "J602" (at 33.02 86.36 0)
+      (effects (font (size 1.27 1.27)))
+    )
+    (property "Value" "12V PWR" (at 33.02 83.82 0)
+      (effects (font (size 1.27 1.27)))
+    )
+    (property "Footprint" "" (at 41.91 83.82 0)
+      (effects (font (size 1.27 1.27)) hide)
+    )
+    (property "Datasheet" "~" (at 41.91 83.82 0)
+      (effects (font (size 1.27 1.27)) hide)
+    )
+    (pin "1")
+    (pin "2")
+    (instances
+      (project "retrofit"
+        (path "/6b7450d6-3952-419a-ab30-dcf88fa68fd4/02d242bf-6dbf-4d5d-8cc6-9f47b3a7e77a"
+          (reference "J602") (unit 1)
+        )
+      )
+    )
+  )
+  (symbol (lib_id "power:GND") (at 46.99 97.79 90) (unit 1)
+    (in_bom yes) (on_board yes) (dnp no)
+    (property "Reference" "#PWR0605" (at 53.34 97.79 0)
+      (effects (font (size 1.27 1.27)) hide)
+    )
+    (property "Value" "GND" (at 49.53 97.79 90)
+      (effects (font (size 1.27 1.27)) (justify right))
+    )
+    (property "Footprint" "" (at 46.99 97.79 0)
+      (effects (font (size 1.27 1.27)) hide)
+    )
+    (property "Datasheet" "" (at 46.99 97.79 0)
+      (effects (font (size 1.27 1.27)) hide)
+    )
+    (pin "1")
+    (instances
+      (project "retrofit"
+        (path "/6b7450d6-3952-419a-ab30-dcf88fa68fd4/02d242bf-6dbf-4d5d-8cc6-9f47b3a7e77a"
+          (reference "#PWR0605") (unit 1)
+        )
+      )
+    )
+  )
+  (symbol (lib_id "power:GND") (at 46.99 86.36 90) (unit 1)
+    (in_bom yes) (on_board yes) (dnp no)
+    (property "Reference" "#PWR0604" (at 53.34 86.36 0)
+      (effects (font (size 1.27 1.27)) hide)
+    )
+    (property "Value" "GND" (at 49.53 86.36 90)
+      (effects (font (size 1.27 1.27)) (justify right))
+    )
+    (property "Footprint" "" (at 46.99 86.36 0)
+      (effects (font (size 1.27 1.27)) hide)
+    )
+    (property "Datasheet" "" (at 46.99 86.36 0)
+      (effects (font (size 1.27 1.27)) hide)
+    )
+    (pin "1")
+    (instances
+      (project "retrofit"
+        (path "/6b7450d6-3952-419a-ab30-dcf88fa68fd4/02d242bf-6dbf-4d5d-8cc6-9f47b3a7e77a"
+          (reference "#PWR0604") (unit 1)
+        )
+      )
+    )
+  )
   (symbol (lib_id "MAHO:ESTOP") (at 129.54 88.9 0) (unit 1)
     (in_bom yes) (on_board yes) (dnp no) (fields_autoplaced)
@@
         )
       )
+    )
+  )
+  (symbol (lib_id "Connector_Generic:Conn_01x02") (at 41.91 95.25 0) (mirror y) (unit 1)
+    (in_bom yes) (on_board yes) (dnp no)
+    (property "Reference" "J603" (at 33.02 97.79 0)
+      (effects (font (size 1.27 1.27)))
+    )
+    (property "Value" "5V PWR" (at 33.02 95.25 0)
+      (effects (font (size 1.27 1.27)))
+    )
+    (property "Footprint" "" (at 41.91 95.25 0)
+      (effects (font (size 1.27 1.27)) hide)
+    )
+    (property "Datasheet" "~" (at 41.91 95.25 0)
+      (effects (font (size 1.27 1.27)) hide)
+    )
+    (pin "1")
+    (pin "2")
+    (instances
+      (project "retrofit"
+        (path "/6b7450d6-3952-419a-ab30-dcf88fa68fd4/02d242bf-6dbf-4d5d-8cc6-9f47b3a7e77a"
+          (reference "J603") (unit 1)
+        )
+      )
