File: schematics/retrofit/Encoders.kicad_sch (KiCad schematic)
At the start: 9 parts, among them U201 LS-403-C, U202 LS-403-C, U203 LS-403-C, U204 EXE-610C, U205 EXE-610C, U206 EXE-610C, U207 7i97-ENC0, U208 7i97-ENC1, U209 7i97-ENC2

Commit message: schematics
Connections:
- net at U206.8 (SHIELD): now also U209.20 (GB2); no longer U203.8 (SHIELD)
- net at U204.2 ((Yellow)_Ie1B): now also U201.2 ((Yellow)_Ie1B)
- net at U204.7 ((Violet)_/Uas): now also U201.7 ((Gray)_Ie0A)
- net at U205.2 ((Yellow)_Ie1B): now also U202.2 ((Yellow)_Ie1B)
- net at U205.7 ((Violet)_/Uas): now also U202.7 ((Gray)_Ie0A)
- net at U205.8 (SHIELD): now also U208.12 (QB1); no longer U202.8 (SHIELD)
- new net: U203.8 (SHIELD), U206.8 (SHIELD)
- new net: U201.8 (SHIELD), U204.8 (SHIELD)
- new net: U202.8 (SHIELD), U205.8 (SHIELD)

Commit message: draft
Connections:
- net at U206.8 (SHIELD): now also U209.20 (GB2); no longer U203.8 (SHIELD)
- net at U204.2 ((Yellow)_Ie1B): now also U201.2 ((Yellow)_Ie1B)
- net at U204.7 ((Violet)_/Uas): now also U201.7 ((Gray)_Ie0A)
- net at U205.2 ((Yellow)_Ie1B): now also U202.2 ((Yellow)_Ie1B)
- net at U205.7 ((Violet)_/Uas): now also U202.7 ((Gray)_Ie0A)
- net at U205.8 (SHIELD): now also U208.12 (QB1); no longer U202.8 (SHIELD)
- new net: U203.8 (SHIELD), U206.8 (SHIELD)
- new net: U201.8 (SHIELD), U204.8 (SHIELD)
- new net: U202.8 (SHIELD), U205.8 (SHIELD)

Commit message: maho-io component and english manual
Parts:
- removed U201, U202, U203: LS-403-C, symbol MAHO:LS-403-C
- removed U204, U205, U206: EXE-610C, symbol MAHO:EXE-610C
- removed U207: 7i97-ENC0, symbol MAHO:7i97-ENC0
- removed U208: 7i97-ENC1, symbol MAHO:7i97-ENC1
- removed U209: 7i97-ENC2, symbol MAHO:7i97-ENC2
Connections:
- no-connect marks 12 -> 0
Other:
- note removed: "BLACK"
- note removed: "BLUE"
- note removed: "BROWN"
- note removed: "GRAY"
- note removed: "GREEN"
- note removed: "PINK"
- note removed: "PINK/GRAY"
- note removed: "PURPLE"
- note removed: "RED"
- note removed: "RED/BLUE"
- note removed: "WHITE"
- note removed: "YELLOW"
