File: schematics/retrofit/LinearEncoders.kicad_sch (KiCad schematic)
At the start: 9 parts, among them U201 LS-403-C, U202 LS-403-C, U203 LS-403-C, U204 EXE-610C, U205 EXE-610C, U206 EXE-610C, U207 7i97-ENC0, U208 7i97-ENC1, U209 7i97-ENC2

Commit message: updates analog
Parts:
- renumbered U205 to EXE?, U206 to EXE?, U204 to EXE?, U201 to LS?, U203 to LS?, U202 to LS?, U207 to U1, U208 to U4, U209 to U7
Connections:
- net at EXE?.2 ((Yellow)_Ie1B): now also LS?.2 ((Yellow)_Ie1B) (x3)
- net at EXE?.7 ((Violet)_/Uas): now also LS?.7 ((Gray)_Ie0A) (x3)
- net at EXE?.8 (SHIELD): now also U1.4 (QB0); no longer LS?.8 (SHIELD)
- new net: EXE?.8 (SHIELD), LS?.8 (SHIELD) (x3)
Changed lines of the file:
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@@
   (symbol (lib_id "MAHO:7i97-ENC2") (at 194.31 132.08 0) (unit 1)
     (in_bom yes) (on_board yes) (dnp no)
-    (property "Reference" "U209" (at 193.04 115.57 0)
+    (property "Reference" "U7" (at 193.04 115.57 0)
       (effects (font (size 1.27 1.27)) (justify left))
     )
@@
   (symbol (lib_name "EXE-610C_2") (lib_id "MAHO:EXE-610C") (at 143.51 93.98 0) (unit 1)
     (in_bom yes) (on_board yes) (dnp no) (fields_autoplaced)
-    (property "Reference" "U205" (at 143.51 113.03 0)
+    (property "Reference" "EXE?" (at 143.51 113.03 0)
       (effects (font (size 1.27 1.27)))
     )
@@
   (symbol (lib_name "EXE-610C_1") (lib_id "MAHO:EXE-610C") (at 143.51 138.43 0) (unit 1)
     (in_bom yes) (on_board yes) (dnp no) (fields_autoplaced)
-    (property "Reference" "U206" (at 143.51 157.48 0)
+    (property "Reference" "EXE?" (at 143.51 157.48 0)
       (effects (font (size 1.27 1.27)))
     )
@@
   (symbol (lib_id "MAHO:7i97-ENC1") (at 194.31 87.63 0) (unit 1)
     (in_bom yes) (on_board yes) (dnp no)
-    (property "Reference" "U208" (at 193.04 71.12 0)
+    (property "Reference" "U4" (at 193.04 71.12 0)
       (effects (font (size 1.27 1.27)) (justify left))
     )
@@
   (symbol (lib_id "MAHO:EXE-610C") (at 143.51 49.53 0) (unit 1)
     (in_bom yes) (on_board yes) (dnp no) (fields_autoplaced)
-    (property "Reference" "U204" (at 143.51 68.58 0)
+    (property "Reference" "EXE?" (at 143.51 68.58 0)
       (effects (font (size 1.27 1.27)))
     )
@@
   (symbol (lib_name "LS-403-C_1") (lib_id "MAHO:LS-403-C") (at 102.87 49.53 0) (unit 1)
     (in_bom yes) (on_board yes) (dnp no) (fields_autoplaced)
-    (property "Reference" "U201" (at 102.87 64.77 0)
+    (property "Reference" "LS?" (at 102.87 64.77 0)
       (effects (font (size 1.27 1.27)))
     )
@@
   (symbol (lib_id "MAHO:LS-403-C") (at 102.87 138.43 0) (unit 1)
     (in_bom yes) (on_board yes) (dnp no) (fields_autoplaced)
-    (property "Reference" "U203" (at 102.87 153.67 0)
+    (property "Reference" "LS?" (at 102.87 153.67 0)
       (effects (font (size 1.27 1.27)))
     )
@@
   (symbol (lib_name "LS-403-C_2") (lib_id "MAHO:LS-403-C") (at 102.87 93.98 0) (unit 1)
     (in_bom yes) (on_board yes) (dnp no) (fields_autoplaced)
-    (property "Reference" "U202" (at 102.87 109.22 0)
+    (property "Reference" "LS?" (at 102.87 109.22 0)
       (effects (font (size 1.27 1.27)))
     )
@@
   (symbol (lib_id "MAHO:7i97-ENC0") (at 194.31 43.18 0) (unit 1)
     (in_bom yes) (on_board yes) (dnp no)
-    (property "Reference" "U207" (at 193.04 26.67 0)
-      (effects (font (size 1.27 1.27)) (justify left))
-    )
+    (property "Reference" "U1" (at 193.04 26.67 0)
+      (effects (font (size 1.27 1.27)) (justify left))
+    )

Commit message: updates
Connections:
- net at EXE?.2 ((Yellow)_Ie1B): now also LS?.2 ((Yellow)_Ie1B) (x3)
- net at EXE?.7 ((Violet)_/Uas): now also LS?.7 ((Gray)_Ie0A) (x3)
- net at EXE?.8 (SHIELD): now also U1.4 (QB0); no longer LS?.8 (SHIELD)
- new net: EXE?.8 (SHIELD), LS?.8 (SHIELD) (x3)

Commit message: updates with new board
Connections:
- net at EXE?.2 ((Yellow)_Ie1B): now also LS?.2 ((Yellow)_Ie1B) (x3)
- net at EXE?.7 ((Violet)_/Uas): now also LS?.7 ((Gray)_Ie0A) (x3)
- net at EXE?.8 (SHIELD): now also U1.4 (QB0); no longer LS?.8 (SHIELD)
- new net: EXE?.8 (SHIELD), LS?.8 (SHIELD) (x3)
