File: schematics/retrofit/retrofit.kicad_sch (KiCad schematic)
At the start: 31 parts, among them J1 PWR, J2 MAHO CTRL, J3 Proximity X, J4 Proximity X, J5 Proximity X, U10 7i97-TB5-Inputs-D, U11 7i97-TB4-Inputs-A, U2 7i97-TB4-RS485, U201 LS-403-C, U202 LS-403-C, U203 LS-403-C, U204 EXE-610C, U205 EXE-610C, U206 EXE-610C, U207 7i97-ENC0, U208 7i97-ENC1, U209 7i97-ENC2, U3 7i97-TB3-ANALOG-A, U5 7i97-TB3-ANALOG-B, U6 7i97-TB3-ANALOG-C, U8 7i97-TB4-Inputs-B, U9 7i97-TB5-Inputs-C

Commit message: sch
Parts:
- removed U201, U202, U203: LS-403-C, symbol MAHO:LS-403-C
- removed U204, U205, U206: EXE-610C, symbol MAHO:EXE-610C
- removed U207: 7i97-ENC0, symbol MAHO:7i97-ENC0
- removed U208: 7i97-ENC1, symbol MAHO:7i97-ENC1
- removed U209: 7i97-ENC2, symbol MAHO:7i97-ENC2
- B?: value (none) -> ~
Connections:
- no-connect marks 36 -> 44
Other:
- removed sheet Encoders
- added sheet Linear Encoders (LinearEncoders.kicad_sch)
- note removed: "BLACK"
- note removed: "BLUE"
- note removed: "BROWN"
- note removed: "GRAY"
- note removed: "GREEN"
- note removed: "PINK"
- note removed: "PINK/GRAY"
- note removed: "PURPLE"
- note removed: "RED"
- note removed: "RED/BLUE"
- note removed: "WHITE"
- note removed: "YELLOW"
- moved on the sheet: J1, J2, J3, J4, J5, J?, U10, U11, U2, U3, U5, U6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

Commit message: updates analog
Connections:
- net at U6.10 (ENA2+): no longer B?. (WHEEL_Z)
- net AN-Z2: now reaches U6.11 (GND)
- net AN-Z2: now also B?. (WHEEL_Z)
- net AN-Z1: now reaches U6.12 (AOUT2)
- net AN-Z1: now also B?. (WHEEL_Z)
- net at U6.9 (ENA2-): no longer B?. (WHEEL_Z)
- net at U5.5 (ENA1-): no longer B?. (WHEEL_Z)
- net at U5.6 (ENA1+): no longer B?. (WHEEL_Z)
- net at U3.1 (ENA0-): no longer B?. (WHEEL_Z)
- net at U3.2 (ENA0+): no longer B?. (WHEEL_Z)
- net AN-Y2: now reaches U5.7 (GND)
- net AN-Y2: now also B?. (WHEEL_Z)
- net AN-Y1: now reaches U5.8 (AOUT1)
- net AN-Y1: now also B?. (WHEEL_Z)
- net AN-X1: now reaches U3.3 (GND)
- net AN-X1: now also B?. (WHEEL_Z)
- net AN-X2: now reaches U3.4 (AOUT0)
- net AN-X2: now also B?. (WHEEL_Z)
Other:
- note added: "BROWN"
- note added: "GRAY"
- note added: "GREEN"
- note added: "PINK"
- note added: "WHITE"
- note added: "YELLOW"
- moved on the sheet: B?

Commit message: updates
Connections:
- net SSG: now reaches B?. (WHEEL_Z), U2.13 (GND)
- net SSG: now also U2.14 (GND)
- net SSTX-: now reaches B?. (WHEEL_Z)
- net SSTX-: now also U2.18 (RS-422/485_RX-); no longer U2.14 (GND)
- net SSRX: now reaches B?. (WHEEL_Z), U2.15 (RS-422/485_RX+)
- net SSRX-: now reaches B?. (WHEEL_Z), U2.16 (RS-422/485_RX-)
- net SSTX: now reaches B?. (WHEEL_Z), U2.17 (RS-422/485_TX+)
- net SS5V: now reaches B?. (WHEEL_Z), U2.19 (5VP)
- net SS5V: now also U2.20 (5VP)
- net O3-: now reaches B?. (WHEEL_Z), U?.19 (OUT3-)
- net O3+: now reaches B?. (WHEEL_Z), U?.20 (OUT3+)
- net O4-: now reaches B?. (WHEEL_Z), U?.21 (OUT4-)
- net O4+: now reaches B?. (WHEEL_Z), U?.22 (OUT4+)
- net O5-: now reaches B?. (WHEEL_Z), U?.23 (OUT5-)
- net O5+: now reaches B?. (WHEEL_Z), U?.24 (OUT5+)
- net I0: now reaches B?. (WHEEL_Z), U11.1 (IN0)
- net I1: now reaches B?. (WHEEL_Z), U11.2 (IN1)
- net CA: now reaches B?. (WHEEL_Z), U11.3 (IN_COMMON_0,1)
- net I2: now reaches B?. (WHEEL_Z), U11.4 (IN2)
- net I3: now reaches B?. (WHEEL_Z), U11.5 (IN3)
- net CB: now reaches B?. (WHEEL_Z), U11.6 (IN_COMMON_2,3)
- net I14: now reaches B?. (WHEEL_Z), U10.10 (IN14)
- net I15: now reaches B?. (WHEEL_Z), U10.11 (IN15)
- net CH: now reaches B?. (WHEEL_Z), U10.12 (IN_COMMON_14,15)
- net I12: now reaches B?. (WHEEL_Z), U10.7 (IN12)
- net I13: now reaches B?. (WHEEL_Z), U10.8 (IN13)
- net CG: now reaches B?. (WHEEL_Z), U10.9 (IN_COMMON_12,13)
- net OO-: now reaches B?. (WHEEL_Z), U?.13 (OUT0-)
- net OO+: now reaches B?. (WHEEL_Z), U?.14 (OUT0+)
- net O1-: now reaches B?. (WHEEL_Z), U?.15 (OUT1-)
- net O1+: now reaches B?. (WHEEL_Z), U?.16 (OUT1+)
- net O2-: now reaches B?. (WHEEL_Z), U?.17 (OUT2-)
- net O2+: now reaches B?. (WHEEL_Z), U?.18 (OUT2+)
- net I6: now reaches B?. (WHEEL_Z), U8.10 (IN6)
- net I7: now reaches B?. (WHEEL_Z), U8.11 (IN7)
- net CD: now reaches B?. (WHEEL_Z), U8.12 (IN_COMMON_6,7)
- net I4: now reaches B?. (WHEEL_Z), U8.7 (IN4)
- net I5: now reaches B?. (WHEEL_Z), U8.8 (IN5)
- net CC: now reaches B?. (WHEEL_Z), U8.9 (IN_COMMON_4,5)
- net I8: now reaches B?. (WHEEL_Z), U9.1 (IN8)
- net I9: now reaches B?. (WHEEL_Z), U9.2 (IN9)
- net CE: now reaches B?. (WHEEL_Z), U9.3 (IN_COMMON_8,9)
- net I10: now reaches B?. (WHEEL_Z), U9.4 (IN10)
- net I11: now reaches B?. (WHEEL_Z), U9.5 (IN11)
- net CF: now reaches B?. (WHEEL_Z), U9.6 (IN_COMMON_10,11)
Other:
- note added: "BLUE"
- note added: "RED"
- moved on the sheet: U10, U11, U2, U3, U5, U6, U8, U9, U?
