File: schematics/maho-io/maho-io.kicad_pcb (KiCad board)
At the start: 2 copper layers, 99.1 x 48.3 mm, 19 parts, among them J1 Conn_01x02, J10 Conn_01x02, J11 Conn_01x02, J2 Conn_01x02, J3 Conn_01x02, J4 Conn_01x02, J5 Conn_01x02, J6 Conn_01x02, J7 Conn_01x02, J8 Conn_01x02, J9 DB37

Commit message: io
Parts:
- added H5: MountingHole, MountingHole:MountingHole_4.5mm, F.Cu at (336.6, 111.9)
- added H6: MountingHole, MountingHole:MountingHole_4.5mm, F.Cu at (336.6, 122.4)
- added J14: LIM_Α_ΙΝ, XY2500R-C(5.08)-3P:XY2500R-C(5.08)-3P, F.Cu at (323.2, 117.1)
- added J29: PWR_ON_INPUTS, XY2500R-C(5.08)-3P:XY2500R-C(5.08)-3P, F.Cu at (323.2, 130.2)
- added J30: PWR_SELECT, Connector_PinSocket_2.54mm:PinSocket_2x03_P2.54mm_Vertical, F.Cu at (363.6, 108.9)
- added J31: PWR, XY2500R-C(5.08)-2P:XY2500R-C(5.08)-2P, F.Cu at (359.4, 64.7)
- added J32: PWR, XY2500R-C(5.08)-2P:XY2500R-C(5.08)-2P, F.Cu at (370.6, 64.7)
- added J33: PWR, XY2500R-C(5.08)-2P:XY2500R-C(5.08)-2P, F.Cu at (336.9, 77.8)
- added J34: PWR, XY2500R-C(5.08)-2P:XY2500R-C(5.08)-2P, F.Cu at (348.1, 77.8)
- added J35: PWR, XY2500R-C(5.08)-2P:XY2500R-C(5.08)-2P, F.Cu at (359.4, 77.8)
- added J36: PWR, XY2500R-C(5.08)-2P:XY2500R-C(5.08)-2P, F.Cu at (370.6, 77.8)
- added J37: PWR, XY2500R-C(5.08)-2P:XY2500R-C(5.08)-2P, F.Cu at (336.9, 90.9)
- added J38: PWR, XY2500R-C(5.08)-2P:XY2500R-C(5.08)-2P, F.Cu at (348.1, 90.9)
- added J39: PWR, XY2500R-C(5.08)-2P:XY2500R-C(5.08)-2P, F.Cu at (359.4, 90.9)
- added J40: PWR, XY2500R-C(5.08)-2P:XY2500R-C(5.08)-2P, F.Cu at (370.6, 90.9)
- added J41: PWR, XY2500R-C(5.08)-2P:XY2500R-C(5.08)-2P, F.Cu at (336.9, 104.0)
- added J42: PWR, XY2500R-C(5.08)-2P:XY2500R-C(5.08)-2P, F.Cu at (348.1, 104.0)
- added J43: PWR, XY2500R-C(5.08)-2P:XY2500R-C(5.08)-2P, F.Cu at (359.4, 104.0)
- added J44: PWR, XY2500R-C(5.08)-2P:XY2500R-C(5.08)-2P, F.Cu at (370.6, 104.0)
- added JJ1: 19X4, Connector_Dsub:DSUB-9_Female_Vertical_P2.77x2.84mm_MountingHoles, F.Cu at (234.2, 109.1)
- added RJ1: SSERIAL, MTJ-88FX1:MTJ-88FX1, F.Cu at (350.3, 117.3)
- J1: value Conn_01x02 -> 19X6_OUTPUTS; footprint TerminalBlock:TerminalBlock_bornier-2_P5.08mm -> Connector_Dsub:DSUB-37_Female_Vertical_P2.77x2.84mm_MountingHoles
- J10: value Conn_01x02 -> ServoY; footprint TerminalBlock:TerminalBlock_bornier-2_P5.08mm -> XY2500R-C(5.08)-2P:XY2500R-C(5.08)-2P
- J11: value Conn_01x02 -> ServoZ; footprint TerminalBlock:TerminalBlock_bornier-2_P5.08mm -> XY2500R-C(5.08)-2P:XY2500R-C(5.08)-2P
- J2: value Conn_01x02 -> 19X7_INPUTS; footprint TerminalBlock:TerminalBlock_bornier-2_P5.08mm -> Connector_Dsub:DSUB-37_Female_Vertical_P2.77x2.84mm_MountingHoles
- J3: value Conn_01x02 -> LIM_X_ΙΝ; footprint TerminalBlock:TerminalBlock_bornier-2_P5.08mm -> XY2500R-C(5.08)-3P:XY2500R-C(5.08)-3P
- J4: value Conn_01x02 -> LIM_Y_ΙΝ; footprint TerminalBlock:TerminalBlock_bornier-2_P5.08mm -> XY2500R-C(5.08)-3P:XY2500R-C(5.08)-3P
- J5: value Conn_01x02 -> LIM_Z_ΙΝ; footprint TerminalBlock:TerminalBlock_bornier-2_P5.08mm -> XY2500R-C(5.08)-3P:XY2500R-C(5.08)-3P
- J6: value Conn_01x02 -> PSU2; footprint TerminalBlock:TerminalBlock_bornier-2_P5.08mm -> XY2500R-C(5.08)-2P:XY2500R-C(5.08)-2P
- J7: value Conn_01x02 -> PSU1; footprint TerminalBlock:TerminalBlock_bornier-2_P5.08mm -> XY2500R-C(5.08)-3P:XY2500R-C(5.08)-3P
- J8: value Conn_01x02 -> PWR; footprint TerminalBlock:TerminalBlock_bornier-2_P5.08mm -> XY2500R-C(5.08)-2P:XY2500R-C(5.08)-2P
- J9: value DB37 -> ServoX; footprint Connector_Dsub:DSUB-37_Female_Horizontal_P2.77x2.84mm_EdgePinOffset7.70mm_Housed_MountingHolesOffset9.12mm -> XY2500R-C(5.08)-2P:XY2500R-C(5.08)-2P
- moved J3 209.0 mm to (323.2, 64.7)
- moved J4 196.6 mm to (323.2, 77.8)
- moved J6 192.6 mm to (336.9, 64.7)
- moved J5 184.9 mm to (323.2, 90.9)
- moved J8 169.2 mm to (348.1, 64.7), turned to 0 degrees
- moved H4 163.4 mm to (29.9, 136.4)
- moved H3 163.0 mm to (237.7, 139.1)
- moved H1 161.4 mm to (29.9, 46.4)
- moved H2 158.8 mm to (237.7, 49.1)
- moved J10 150.9 mm to (239.7, 75.9)
- moved J11 150.8 mm to (239.7, 87.1)
- moved J7 143.1 mm to (323.2, 104.0), turned to 0 degrees
- moved J9 130.7 mm to (239.7, 64.7), turned to -90 degrees
- moved R2 110.8 mm to (252.0, 142.1), turned to 0 degrees
- moved R1 104.4 mm to (252.0, 138.0), turned to 0 degrees
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Connections:
- J1 pad 1: GND -> /19X6_HANDWHEEL_X
- J1 pad 2: GND -> /19X6_HANDWHEEL_Z
- J10 pad 1: Earth -> /E301
- J10 pad 2: GND -> /E302
- J11 pad 1: GND -> /E201
- J11 pad 2: GND -> /E202
- J2 pad 1: GND -> /19X7_HANDWHEEL_X
- J2 pad 2: /P1 -> /19X7_HANDWHEEL_Y
- J3 pad 1: /P2 -> GND
- J3 pad 2: /P3 -> /LIMIT_X
- J4 pad 1: /P4 -> GND
- J4 pad 2: /P5 -> /LIMIT_Υ
- J5 pad 1: /P6 -> GND
- J5 pad 2: /P7 -> /LIMIT_Ζ
- J6 pad 1: /P8 -> /202_24V
- J6 pad 2: /P34 -> GND
- J7 pad 1: /24V -> /200_NORMAL
- J7 pad 2: /24V -> GND
- J8 pad 1: /24V/a -> /EXT_PWR
- J8 pad 2: /24V/a -> GND
- J9 pad 1: /P1 -> /E101
- J9 pad 2: /P2 -> /E102
- R1 pad 1: /24V -> /EXT_PWR
- R2 pad 1: /24V/a -> /204_24V/a
Routing:
- net GND: track 111.3 -> 0.00 mm
- net Earth: track 94.1 -> 0.00 mm
- net /P8: track 42.8 -> 0.00 mm
- net /P7: track 41.9 -> 0.00 mm
- net /P6: track 40.9 -> 0.00 mm
- net /P5: track 40.0 -> 0.00 mm
- net /P34: track 39.2 -> 0.00 mm
- net /P4: track 39.0 -> 0.00 mm
- net /P3: track 38.0 -> 0.00 mm
- net /P2: track 37.1 -> 0.00 mm
- net /P1: track 36.1 -> 0.00 mm
- net /24V/a: track 31.2 -> 0.00 mm
- net /24V: track 29.4 -> 0.00 mm
- net Net-(D1-A): track 17.1 -> 0.00 mm
- net Net-(D2-A): track 16.3 -> 0.00 mm
- removed copper zone on B.Cu, net GND
Other:
- board outline removed
- board text removed: "24V"
- board text removed: "24V/a"
- board text removed: "EARTH"
- board text removed: "GND"
- board text removed: "P1"
- board text removed: "P2"
- board text removed: "P3"
- board text removed: "P34"
- board text removed: "P4"
- board text removed: "P5"
- board text removed: "P6"
- board text removed: "P7"
- board text removed: "P8"

Commit message: maho-io
Parts:
- removed J10: ServoY, XY2500R-C(5.08)-2P:XY2500R-C(5.08)-2P
- removed J11: ServoZ, XY2500R-C(5.08)-2P:XY2500R-C(5.08)-2P
- removed J9: ServoX, XY2500R-C(5.08)-2P:XY2500R-C(5.08)-2P
- added U1: ~, XY2500V-C(5.08)-2P:XY2500V-C(5.08)-2P, F.Cu at (80.5, 111.4)
- added U10: ~, XY2500V-C(5.08)-2P:XY2500V-C(5.08)-2P, F.Cu at (91.8, 146.7)
- added U11: ~, XY2500V-C(5.08)-2P:XY2500V-C(5.08)-2P, F.Cu at (103.0, 146.7)
- added U12: ~, XY2500V-C(5.08)-3P:XY2500V-C(5.08)-3P, F.Cu at (83.0, 76.1)
- added U13: ~, XY2500V-C(5.08)-3P:XY2500V-C(5.08)-3P, F.Cu at (99.4, 76.1)
- added U14: ~, XY2500V-C(5.08)-3P:XY2500V-C(5.08)-3P, F.Cu at (115.7, 76.1)
- added U15: ~, XY2500V-C(5.08)-3P:XY2500V-C(5.08)-3P, F.Cu at (132.1, 76.1)
- added U16: ~, XY2500V-C(5.08)-3P:XY2500V-C(5.08)-3P, F.Cu at (83.0, 93.8)
- added U17: ~, XY2500V-C(5.08)-3P:XY2500V-C(5.08)-3P, F.Cu at (99.4, 93.8)
- added U18: ~, XY2500V-C(5.08)-3P:XY2500V-C(5.08)-3P, F.Cu at (115.7, 93.8)
- added U19: ~, XY2500V-C(5.08)-4P:XY2500V-C(5.08)-4P, F.Cu at (175.5, 111.4)
- added U2: ~, XY2500V-C(5.08)-2P:XY2500V-C(5.08)-2P, F.Cu at (91.8, 111.4)
- added U20: ~, XY2500V-C(5.08)-4P:XY2500V-C(5.08)-4P, F.Cu at (175.5, 129.0)
- added U21: ~, XY2500V-C(5.08)-2P:XY2500V-C(5.08)-2P, F.Cu at (114.3, 146.7)
- added U3: ~, XY2500V-C(5.08)-2P:XY2500V-C(5.08)-2P, F.Cu at (103.0, 111.4)
- added U4: ~, XY2500V-C(5.08)-2P:XY2500V-C(5.08)-2P, F.Cu at (114.3, 111.4)
- added U5: ~, XY2500V-C(5.08)-2P:XY2500V-C(5.08)-2P, F.Cu at (80.5, 129.0)
- added U6: ~, XY2500V-C(5.08)-2P:XY2500V-C(5.08)-2P, F.Cu at (91.8, 129.0)
- added U7: ~, XY2500V-C(5.08)-2P:XY2500V-C(5.08)-2P, F.Cu at (103.0, 129.0)
- added U8: ~, XY2500V-C(5.08)-2P:XY2500V-C(5.08)-2P, F.Cu at (114.3, 129.0)
- added U9: ~, XY2500V-C(5.08)-2P:XY2500V-C(5.08)-2P, F.Cu at (80.5, 146.7)
- moved J14 257.4 mm to (66.7, 95.8)
- moved J29 257.4 mm to (66.7, 108.9)
- moved J3 257.4 mm to (66.7, 43.3)
- moved J4 257.4 mm to (66.7, 56.4)
- moved J5 257.4 mm to (66.7, 69.5)
- moved J7 257.4 mm to (66.7, 82.6)
- moved J31 215.9 mm to (147.9, 108.7)
- moved J35 215.9 mm to (147.9, 121.8)
- moved J39 215.9 mm to (147.9, 134.9)
- moved J43 215.9 mm to (147.9, 148.0)
- moved J32 215.9 mm to (159.2, 108.7)
- moved J36 215.9 mm to (159.2, 121.8)
- moved J40 215.9 mm to (159.2, 134.9)
- moved J44 215.9 mm to (159.2, 148.0)
- moved J33 215.9 mm to (125.5, 121.8)
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
Commit message: maho-io
Parts:
- removed J14: LIM_Α_ΙΝ, XY2500R-C(5.08)-3P:XY2500R-C(5.08)-3P
- removed J29: PWR_ON_INPUTS, XY2500R-C(5.08)-3P:XY2500R-C(5.08)-3P
- removed J30: PWR_SELECT, Connector_PinSocket_2.54mm:PinSocket_2x03_P2.54mm_Vertical
- removed J31, J32, J33, J34, J35, J36, J37, J38, J39, J40, J41, J42, J43, J44, J8: PWR, XY2500R-C(5.08)-2P:XY2500R-C(5.08)-2P
- removed J4: LIM_Y_ΙΝ, XY2500R-C(5.08)-3P:XY2500R-C(5.08)-3P
- removed J5: LIM_Z_ΙΝ, XY2500R-C(5.08)-3P:XY2500R-C(5.08)-3P
- removed J6: PSU2, XY2500R-C(5.08)-2P:XY2500R-C(5.08)-2P
- removed J7: PSU1, XY2500R-C(5.08)-3P:XY2500R-C(5.08)-3P
- removed JJ1: 19X4, Connector_Dsub:DSUB-9_Female_Vertical_P2.77x2.84mm_MountingHoles
- removed U1, U10, U11, U2, U21, U3, U4, U5, U6, U7, U8, U9: ~, XY2500V-C(5.08)-2P:XY2500V-C(5.08)-2P
- removed U12, U13, U14, U15, U16, U17, U18: ~, XY2500V-C(5.08)-3P:XY2500V-C(5.08)-3P
- removed U19, U20: ~, XY2500V-C(5.08)-4P:XY2500V-C(5.08)-4P
- added A1: 19X4, Connector_Dsub:DSUB-9_Female_Vertical_P2.77x2.84mm_MountingHoles, F.Cu at (219.5, 112.6)
- added D3: LED, LED_THT:LED_D5.0mm, F.Cu at (190.4, 128.0)
- added DBI1: 19X7_INPUTS, Connector_Dsub:DSUB-37_Female_Vertical_P2.77x2.84mm_MountingHoles, F.Cu at (96.2, 59.1)
- added DBO1: 19X6_OUTPUTS, Connector_Dsub:DSUB-37_Female_Vertical_P2.77x2.84mm_MountingHoles, F.Cu at (76.9, 59.2)
- added E1: Chassis, MountingHole:MountingHole_4.5mm_Pad, F.Cu at (89.9, 129.9)
- added G1: G, XY2500V-C(5.08)-2P:XY2500V-C(5.08)-2P, F.Cu at (176.2, 86.8)
- added G2: G, XY2500V-C(5.08)-2P:XY2500V-C(5.08)-2P, F.Cu at (176.2, 96.9)
- added G3: G, XY2500V-C(5.08)-2P:XY2500V-C(5.08)-2P, F.Cu at (176.2, 107.1)
- added GA1: GA, XY2500V-C(5.08)-2P:XY2500V-C(5.08)-2P, F.Cu at (195.9, 71.5)
- added GA2: GA, XY2500V-C(5.08)-2P:XY2500V-C(5.08)-2P, F.Cu at (195.9, 81.7)
- added GA3: GA, XY2500V-C(5.08)-2P:XY2500V-C(5.08)-2P, F.Cu at (195.9, 91.8)
- added IN1: IN1, XY2500V-C(5.08)-3P:XY2500V-C(5.08)-3P, F.Cu at (134.3, 63.9)
- added IN2: IN2, XY2500V-C(5.08)-3P:XY2500V-C(5.08)-3P, F.Cu at (154.6, 43.6)
- added IN3: IN3, XY2500V-C(5.08)-3P:XY2500V-C(5.08)-3P, F.Cu at (154.6, 58.8)
- added IN4: IN4, XY2500V-C(5.08)-3P:XY2500V-C(5.08)-3P, F.Cu at (134.3, 79.2)
- added IN5: IN5, XY2500V-C(5.08)-3P:XY2500V-C(5.08)-3P, F.Cu at (134.3, 94.4)
- added IN6: IN6, XY2500V-C(5.08)-3P:XY2500V-C(5.08)-3P, F.Cu at (134.3, 109.6)
- added IN7: IN7, XY2500V-C(5.08)-3P:XY2500V-C(5.08)-3P, F.Cu at (134.3, 124.9)
- added JP1: PWR_SELECT, Connector_PinSocket_2.54mm:PinSocket_2x03_P2.54mm_Vertical, F.Cu at (200.4, 128.7)
- added JP2: GND_BRIGDE, Connector_PinSocket_2.54mm:PinSocket_2x03_P2.54mm_Vertical, F.Cu at (205.4, 121.1)
- added L1: LIM, XY2500V-C(5.08)-3P:XY2500V-C(5.08)-3P, F.Cu at (154.6, 74.1)
- added L2: LIM, XY2500V-C(5.08)-3P:XY2500V-C(5.08)-3P, F.Cu at (154.6, 89.3)
- added L3: LIM, XY2500V-C(5.08)-3P:XY2500V-C(5.08)-3P, F.Cu at (154.6, 104.5)
- added L4: LIM, XY2500V-C(5.08)-3P:XY2500V-C(5.08)-3P, F.Cu at (154.6, 119.8)
- added OUT1: OUT1, XY2500V-C(5.08)-2P:XY2500V-C(5.08)-2P, F.Cu at (115.3, 41.0)
- added OUT2: OUT2, XY2500V-C(5.08)-2P:XY2500V-C(5.08)-2P, F.Cu at (115.3, 51.2)
- added OUT3: OUT3, XY2500V-C(5.08)-2P:XY2500V-C(5.08)-2P, F.Cu at (115.3, 61.4)
- added OUT34: OUT34, XY2500V-C(5.08)-2P:XY2500V-C(5.08)-2P, F.Cu at (115.3, 122.3)
- added OUT4: OUT4, XY2500V-C(5.08)-2P:XY2500V-C(5.08)-2P, F.Cu at (115.3, 71.5)
- added OUT5: OUT5, XY2500V-C(5.08)-2P:XY2500V-C(5.08)-2P, F.Cu at (115.3, 81.7)
- added OUT6: OUT6, XY2500V-C(5.08)-2P:XY2500V-C(5.08)-2P, F.Cu at (115.3, 91.8)
- added OUT7: OUT7, XY2500V-C(5.08)-2P:XY2500V-C(5.08)-2P, F.Cu at (115.3, 102.0)
- added OUT8: OUT8, XY2500V-C(5.08)-2P:XY2500V-C(5.08)-2P, F.Cu at (115.3, 112.2)
- added PON1: POWER_ON_SWITCHES, XY2500V-C(5.08)-4P:XY2500V-C(5.08)-4P, F.Cu at (134.3, 46.1)
- added R3: R, Resistor_SMD:R_0805_2012Metric, F.Cu at (189.2, 132.5)
- added S1: S1, XY2500V-C(5.08)-2P:XY2500V-C(5.08)-2P, F.Cu at (237.2, 95.7)
- added S2: S2, XY2500V-C(5.08)-2P:XY2500V-C(5.08)-2P, F.Cu at (237.2, 105.8)
- added S3: S3, XY2500V-C(5.08)-2P:XY2500V-C(5.08)-2P, F.Cu at (237.2, 116.0)
- added SS1: SS1, XY2500V-C(5.08)-4P:XY2500V-C(5.08)-4P, F.Cu at (237.2, 60.1)
- added SS2: SS2, XY2500V-C(5.08)-4P:XY2500V-C(5.08)-4P, F.Cu at (237.2, 80.4)
- added V1: V, XY2500V-C(5.08)-2P:XY2500V-C(5.08)-2P, F.Cu at (176.2, 56.3)
- added V2: V, XY2500V-C(5.08)-2P:XY2500V-C(5.08)-2P, F.Cu at (176.2, 66.5)
- added V3: V, XY2500V-C(5.08)-2P:XY2500V-C(5.08)-2P, F.Cu at (176.2, 76.6)
- added VA1: VA, XY2500V-C(5.08)-2P:XY2500V-C(5.08)-2P, F.Cu at (195.9, 41.0)
- added VA2: VA, XY2500V-C(5.08)-2P:XY2500V-C(5.08)-2P, F.Cu at (195.9, 51.2)
- added VA3: VA, XY2500V-C(5.08)-2P:XY2500V-C(5.08)-2P, F.Cu at (195.9, 61.4)
- J1: value 19X6_OUTPUTS -> PWR; footprint Connector_Dsub:DSUB-37_Female_Vertical_P2.77x2.84mm_MountingHoles -> XY2500V-C(5.08)-2P:XY2500V-C(5.08)-2P
- J2: value 19X7_INPUTS -> V2; footprint Connector_Dsub:DSUB-37_Female_Vertical_P2.77x2.84mm_MountingHoles -> XY2500V-C(5.08)-2P:XY2500V-C(5.08)-2P
- J3: value LIM_X_ΙΝ -> V1; footprint XY2500R-C(5.08)-3P:XY2500R-C(5.08)-3P -> XY2500V-C(5.08)-3P:XY2500V-C(5.08)-3P
- R1, R2: footprint Resistor_THT:R_Axial_DIN0207_L6.3mm_D2.5mm_P10.16mm_Horizontal -> Resistor_SMD:R_0805_2012Metric
- moved H6 125.6 mm to (77.1, 130.0)
- moved H4 110.7 mm to (237.1, 130.0)
- moved J3 109.5 mm to (176.2, 43.6), turned to -90 degrees
- moved H5 92.2 mm to (167.1, 130.0)
- moved J1 88.1 mm to (176.2, 117.2), turned to -90 degrees
- moved RJ1 83.0 mm to (220.7, 47.4)
- moved J2 77.1 mm to (195.9, 102.0), turned to -90 degrees
- moved H3 75.0 mm to (237.1, 40.0)
- moved H1 74.5 mm to (77.1, 40.0)
- moved D1 52.1 mm to (183.4, 128.0), turned to 180 degrees
- moved R1 48.8 mm to (182.2, 132.5), turned to 180 degrees
- moved D2 47.3 mm to (176.5, 128.0), turned to 180 degrees
- moved R2 42.3 mm to (175.3, 132.5), turned to 180 degrees
- moved H2 17.7 mm to (167.1, 40.0)
Connections:
- J1 pad 1: /19X6_HANDWHEEL_X -> /EXT_PWR
- J1 pad 2: /19X6_HANDWHEEL_Z -> GND
- J2 pad 1: /19X7_HANDWHEEL_X -> /202_24V
- J2 pad 2: /19X7_HANDWHEEL_Y -> GNDA
- J3 pad 1: GND -> /204_24V/a
- J3 pad 2: /LIMIT_X -> /200_NORMAL
- J3 pad 3: VDC -> GND
- RJ1 pad 1: Net-(RJ1-Pad1) -> /SS_TX-
- RJ1 pad 2: Net-(RJ1-Pad2) -> /SS_TX+
- RJ1 pad 3: Net-(RJ1-Pad3) -> /SS_RX-
- RJ1 pad 4: Net-(RJ1-Pad4) -> GND
- RJ1 pad 5: Net-(RJ1-Pad5) -> GND
- RJ1 pad 6: Net-(RJ1-Pad6) -> /SS_RX+
- RJ1 pad 7: Net-(RJ1-Pad7) -> /SS_5VP
- RJ1 pad 8: Net-(RJ1-Pad8) -> /SS_5VP
Other:
- board outline added: 170 x 100 mm
- board text added: "SSERIAL NEEDS PINOUT VALIDATION"
