File: schematics/maho-io/maho-io.kicad_sch (KiCad schematic)
At the start: 17 parts, among them J1 19X6_OUTPUTS, J2 19X7_INPUTS, J4 LIMIT_X, J5 LIMIT_Y, J6 LIMIT_Z, J7 Conn_01x02, J8 X10, J9 Conn_01x02

Commit message: io
Parts:
- added H5, H6: MountingHole, MountingHole:MountingHole_4.5mm, symbol Mechanical:MountingHole
- added J10: SERVO_Y, symbol Connector_Generic:Conn_01x02
- added J11: SERVO_Z, symbol Connector_Generic:Conn_01x02
- added J12: OUTPUT_1, symbol Connector_Generic:Conn_01x02
- added J13: OUTPUT_2, symbol Connector_Generic:Conn_01x02
- added J14: LIM_Α_ΙΝ, XY2500R-C(5.08)-3P:XY2500R-C(5.08)-3P, symbol Connector_Generic:Conn_01x03
- added J15: OUTPUT_3, symbol Connector_Generic:Conn_01x02
- added J16: OUTPUT_4, symbol Connector_Generic:Conn_01x02
- added J17: OUTPUT_5, symbol Connector_Generic:Conn_01x02
- added J18: OUTPUT_6, symbol Connector_Generic:Conn_01x02
- added J19: OUTPUT_7, symbol Connector_Generic:Conn_01x02
- added J20: OUTPUT_8, symbol Connector_Generic:Conn_01x02
- added J21: INPUT_1, symbol Connector_Generic:Conn_01x03
- added J22, J26: INPUT_2, symbol Connector_Generic:Conn_01x03
- added J23, J27: INPUT_3, symbol Connector_Generic:Conn_01x03
- added J24: INPUT_4, symbol Connector_Generic:Conn_01x03
- added J25: INPUT_5, symbol Connector_Generic:Conn_01x03
- added J28: OUTPUT_34, symbol Connector_Generic:Conn_01x02
- added J29: PWR_ON_INPUTS, XY2500R-C(5.08)-3P:XY2500R-C(5.08)-3P, symbol Connector_Generic:Conn_01x03
- added J30: PWR_SELECT, Connector_PinSocket_2.54mm:PinSocket_2x03_P2.54mm_Vertical, symbol Connector_Generic:Conn_02x03_Odd_Even
- added J31, J32, J33, J34, J35, J36, J37, J38, J39, J40, J41, J42, J43, J44: PWR, XY2500R-C(5.08)-2P:XY2500R-C(5.08)-2P, symbol Connector_Generic:Conn_01x02
- added J45: Chassis, symbol Connector_Generic:Conn_01x01
- added J46: SSERIAL_A, symbol Connector_Generic:Conn_01x04
- added J47: SSERIAL_B, symbol Connector_Generic:Conn_01x04
- added J9: SERVO_X, symbol Connector_Generic:Conn_01x02
- added RJ1: SSERIAL, MTJ-88FX1:MTJ-88FX1, symbol MTJ-88FX1:MTJ-88FX1
- J1, J2: footprint Connector_Dsub:DSUB-37_Female_Horizontal_P2.77x2.84mm_EdgePinOffset7.70mm_Housed_MountingHolesOffset9.12mm -> Connector_Dsub:DSUB-37_Female_Vertical_P2.77x2.84mm_MountingHoles
- J3: renamed from J4; value LIMIT_X -> LIM_X_ΙΝ; footprint (none) -> XY2500R-C(5.08)-3P:XY2500R-C(5.08)-3P
- J4: renamed from J5; value LIMIT_Y -> LIM_Y_ΙΝ; footprint (none) -> XY2500R-C(5.08)-3P:XY2500R-C(5.08)-3P
- J5: renamed from J6; value LIMIT_Z -> LIM_Z_ΙΝ; footprint (none) -> XY2500R-C(5.08)-3P:XY2500R-C(5.08)-3P
- J6: renamed from J7; value Conn_01x02 -> PSU2; footprint (none) -> XY2500R-C(5.08)-2P:XY2500R-C(5.08)-2P
- J7: renamed from J8; value X10 -> PSU1; footprint (none) -> XY2500R-C(5.08)-3P:XY2500R-C(5.08)-3P
- J8: renamed from J9; value Conn_01x02 -> PWR; footprint (none) -> XY2500R-C(5.08)-2P:XY2500R-C(5.08)-2P
- JJ1: renamed from JJ3; footprint (none) -> Connector_Dsub:DSUB-9_Female_Vertical_P2.77x2.84mm_MountingHoles
- renumbered D3 to D1, D4 to D2, R3 to R1, R4 to R2
Connections:
- net 201_0V is gone; now on net GND: J7.2 (Pin_2)
- net 203_0V is gone; now on net GND: J6.2 (Pin_2)
- net 200_NORMAL: now also J12.1 (Pin_1), J13.1 (Pin_1), J15.1 (Pin_1), J16.1 (Pin_1), J17.1 (Pin_1), J18.1 (Pin_1), J19.1 (Pin_1), J20.1 (Pin_1)
- net 204_24V/a: now also R2.1, J30.5 (Pin_5), J30.6 (Pin_6)
- net EXT_PWR: now also R1.1, J30.1 (Pin_1), J30.2 (Pin_2)
- net Earth: now also J45.1 (Pin_1)
- net GND: now also J14.1 (Pin_1), J21.3 (Pin_3), J22.3 (Pin_3), J23.3 (Pin_3), J24.3 (Pin_3), J25.3 (Pin_3), J26.3 (Pin_3), J27.3 (Pin_3), J31.1 (Pin_1), J31.2 (Pin_2), J32.1 (Pin_1), J32.2 (Pin_2), J33.1 (Pin_1), J33.2 (Pin_2), J34.1 (Pin_1), J34.2 (Pin_2), J35.1 (Pin_1), J35.2 (Pin_2), J36.1 (Pin_1), J36.2 (Pin_2), J37.1 (Pin_1), J37.2 (Pin_2)
- net LIMIT_X: now also J26.1 (Pin_1); no longer J4.2 (Pin_2), J5.2 (Pin_2)
- net VDC: now also J14.3 (Pin_3), J28.1 (Pin_1), J29.1 (Pin_1), J30.3 (Pin_3), J30.4 (Pin_4), J38.1 (Pin_1), J38.2 (Pin_2), J39.1 (Pin_1), J39.2 (Pin_2), J40.1 (Pin_1), J40.2 (Pin_2), J41.1 (Pin_1), J41.2 (Pin_2), J42.1 (Pin_1), J42.2 (Pin_2), J43.1 (Pin_1), J43.2 (Pin_2), J44.1 (Pin_1), J44.2 (Pin_2)
- net E101: now reaches JJ1.1
- net E101: now also J9.1 (Pin_1)
- net E102: now reaches JJ1.2
- net E102: now also J9.2 (Pin_2)
- net E201: now reaches JJ1.3
- net E201: now also J11.1 (Pin_1)
- net E202: now reaches JJ1.4
- net E202: now also J11.2 (Pin_2)
- net E301: now reaches JJ1.5
- net E301: now also J10.1 (Pin_1)
- net E302: now reaches JJ1.9
- net E302: now also J10.2 (Pin_2)
- net P1 renamed 19X6_HANDWHEEL_X
- net 19X6_HANDWHEEL_X: now also J12.2 (Pin_2); no longer J2.1
- net P2 renamed 19X6_HANDWHEEL_Z
- net 19X6_HANDWHEEL_Z: now also J15.2 (Pin_2); no longer J2.2
- net P3 renamed 19X6_HANDWHEEL_Y
- net 19X6_HANDWHEEL_Y: now also J13.2 (Pin_2); no longer J2.3
- net P34: no longer names the net of J2.34
- net P34: no longer J1.34
- net P4 renamed 19X7_24V
- net 19X7_24V: now also J23.2 (Pin_2); no longer J1.4
- net P5 renamed 19X7_MAIN_DRIVE_OFF
- net 19X7_MAIN_DRIVE_OFF: now also J24.1 (Pin_1); no longer J1.5
- net P6 renamed 19X7_NOT_SPINDLE_FEED
- net 19X7_NOT_SPINDLE_FEED: now also J24.2 (Pin_2); no longer J1.6
- net P7 renamed 19X7_LUBRICANT
- net 19X7_LUBRICANT: now also J25.1 (Pin_1); no longer J1.7
- net P8: no longer names the net of J2.8
- net P8: no longer J1.8
- new net: J46.1 (Pin_1), RJ1.1
- new net: J46.2 (Pin_2), RJ1.2
- new net: J46.3 (Pin_3), RJ1.3
- new net: J46.4 (Pin_4), RJ1.4
- new net: J47.1 (Pin_1), RJ1.5
- new net: J47.2 (Pin_2), RJ1.6
- new net: J47.3 (Pin_3), RJ1.7
- new net: J47.4 (Pin_4), RJ1.8
- new net 19X7_HANDWHEEL_X: J2.1, J22.1 (Pin_1)
- new net 19X7_HANDWHEEL_Y: J2.2, J22.2 (Pin_2)
- new net 19X7_HANDWHEEL_Z: J2.3, J23.1 (Pin_1)
- new net CENTRAL_LUBRICATION: J1.8, J20.2 (Pin_2)
- new net COOLANT_PUMP: J1.6, J18.2 (Pin_2)
- new net EXTERNAL_ESTOP: J21.1 (Pin_1), J29.3 (Pin_3)
- new net LIMIT_Α: J14.2 (Pin_2), J27.2 (Pin_2)
- new net LIMIT_Ζ: J27.1 (Pin_1), J5.2 (Pin_2)
- new net LIMIT_Υ: J26.2 (Pin_2), J4.2 (Pin_2)
- new net POWER_SWITCH: J21.2 (Pin_2), J29.2 (Pin_2)
- new net SPINDLE_CCW: J1.5, J17.2 (Pin_2)
- new net SPINDLE_CW: J1.4, J16.2 (Pin_2)
- new net TOOL_RELEASE: J1.7, J19.2 (Pin_2)
- new net /ESTOP: J1.34, J28.2 (Pin_2)
- no-connect marks 56 -> 62
Other:
- note added: "200"
- note added: "201"
- note added: "202"
- note added: "203"
- note added: "204"
- moved on the sheet: D1, D2, H1, H2, H3, H4, J1, J2, J3, J4, J5, J6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

Commit message: maho-io
Parts:
- removed J10: SERVO_Y, symbol Connector_Generic:Conn_01x02
- removed J11: SERVO_Z, symbol Connector_Generic:Conn_01x02
- removed J12: OUTPUT_1, symbol Connector_Generic:Conn_01x02
- removed J13: OUTPUT_2, symbol Connector_Generic:Conn_01x02
- removed J15: OUTPUT_3, symbol Connector_Generic:Conn_01x02
- removed J16: OUTPUT_4, symbol Connector_Generic:Conn_01x02
- removed J17: OUTPUT_5, symbol Connector_Generic:Conn_01x02
- removed J18: OUTPUT_6, symbol Connector_Generic:Conn_01x02
- removed J19: OUTPUT_7, symbol Connector_Generic:Conn_01x02
- removed J20: OUTPUT_8, symbol Connector_Generic:Conn_01x02
- removed J21: INPUT_1, symbol Connector_Generic:Conn_01x03
- removed J22, J26: INPUT_2, symbol Connector_Generic:Conn_01x03
- removed J23, J27: INPUT_3, symbol Connector_Generic:Conn_01x03
- removed J24: INPUT_4, symbol Connector_Generic:Conn_01x03
- removed J25: INPUT_5, symbol Connector_Generic:Conn_01x03
- removed J28: OUTPUT_34, symbol Connector_Generic:Conn_01x02
- removed J46: SSERIAL_A, symbol Connector_Generic:Conn_01x04
- removed J47: SSERIAL_B, symbol Connector_Generic:Conn_01x04
- removed J9: SERVO_X, symbol Connector_Generic:Conn_01x02
- added U1, U10, U11, U2, U21, U3, U4, U5, U6, U7, U8, U9: ~, XY2500V-C(5.08)-2P:XY2500V-C(5.08)-2P, symbol XY2500V-C(5.08)-2P:XY2500V-C(5.08)-2P
- added U12, U13, U14, U15, U16, U17, U18: ~, XY2500V-C(5.08)-3P:XY2500V-C(5.08)-3P, symbol XY2500V-C(5.08)-3P:XY2500V-C(5.08)-3P
- added U19, U20: ~, XY2500V-C(5.08)-4P:XY2500V-C(5.08)-4P, symbol XY2500V-C(5.08)-4P:XY2500V-C(5.08)-4P
Connections:
- net 19X6_HANDWHEEL_X: now also U1.2
- net 19X6_HANDWHEEL_Y: now also U2.2
- net 19X6_HANDWHEEL_Z: now also U3.2
- net 19X7_24V: now also U14.2
- net 19X7_HANDWHEEL_X: now also U13.1
- net 19X7_HANDWHEEL_Y: now also U13.2
- net 19X7_HANDWHEEL_Z: now also U14.1
- net 19X7_LUBRICANT: now also U16.1
- net 19X7_MAIN_DRIVE_OFF: now also U15.1
- net 19X7_NOT_SPINDLE_FEED: now also U15.2
- net 200_NORMAL: now also U1.1, U2.1, U3.1, U4.1, U5.1, U6.1, U7.1, U8.1
- net CENTRAL_LUBRICATION: now also U8.2
- net COOLANT_PUMP: now also U6.2
- net E101: now also U9.1
- net E102: now also U9.2
- net E201: now also U11.1
- net E202: now also U11.2
- net E301: now also U10.1
- net E302: now also U10.2
- net EXTERNAL_ESTOP: now also U12.1
- net GND: now also U12.3, U13.3, U14.3, U15.3, U16.3, U17.3, U18.3
- net LIMIT_X: now also U17.1
- net LIMIT_Α: now also U18.2
- net LIMIT_Ζ: now also U18.1
- net LIMIT_Υ: now also U17.2
- net POWER_SWITCH: now also U12.2
- net SPINDLE_CCW: now also U5.2
- net SPINDLE_CW: now also U4.2
- net TOOL_RELEASE: now also U7.2
- net VDC: now also U21.1
- net /ESTOP: now also U21.2
- net at RJ1.1: now also U19.1
- net at RJ1.2: now also U19.2
- net at RJ1.3: now also U19.3
- net at RJ1.4: now also U19.4
- net at RJ1.5: now also U20.1
- net at RJ1.6: now also U20.2
- net at RJ1.7: now also U20.3
- net at RJ1.8: now also U20.4

Commit message: maho-io
Parts:
- removed J14: LIM_Α_ΙΝ, XY2500R-C(5.08)-3P:XY2500R-C(5.08)-3P, symbol Connector_Generic:Conn_01x03
- removed J29: PWR_ON_INPUTS, XY2500R-C(5.08)-3P:XY2500R-C(5.08)-3P, symbol Connector_Generic:Conn_01x03
- removed J3: LIM_X_ΙΝ, XY2500R-C(5.08)-3P:XY2500R-C(5.08)-3P, symbol Connector_Generic:Conn_01x03
- removed J31, J32, J33, J34, J35, J36, J37, J38, J39, J40, J41, J42, J43, J44, J8: PWR, XY2500R-C(5.08)-2P:XY2500R-C(5.08)-2P, symbol Connector_Generic:Conn_01x02
- removed J4: LIM_Y_ΙΝ, XY2500R-C(5.08)-3P:XY2500R-C(5.08)-3P, symbol Connector_Generic:Conn_01x03
- removed J5: LIM_Z_ΙΝ, XY2500R-C(5.08)-3P:XY2500R-C(5.08)-3P, symbol Connector_Generic:Conn_01x03
- removed J6: PSU2, XY2500R-C(5.08)-2P:XY2500R-C(5.08)-2P, symbol Connector_Generic:Conn_01x02
- removed J7: PSU1, XY2500R-C(5.08)-3P:XY2500R-C(5.08)-3P, symbol Connector_Generic:Conn_01x03
- added D3: LED, LED_THT:LED_D5.0mm, symbol Device:LED
- added G1, G2, G3: G, XY2500V-C(5.08)-2P:XY2500V-C(5.08)-2P, symbol XY2500V-C(5.08)-2P:XY2500V-C(5.08)-2P
- added GA1, GA2, GA3: GA, XY2500V-C(5.08)-2P:XY2500V-C(5.08)-2P, symbol XY2500V-C(5.08)-2P:XY2500V-C(5.08)-2P
- added J1: PWR, XY2500V-C(5.08)-2P:XY2500V-C(5.08)-2P, symbol XY2500V-C(5.08)-2P:XY2500V-C(5.08)-2P
- added J2: V2, XY2500V-C(5.08)-2P:XY2500V-C(5.08)-2P, symbol XY2500V-C(5.08)-2P:XY2500V-C(5.08)-2P
- added J3: V1, XY2500V-C(5.08)-3P:XY2500V-C(5.08)-3P, symbol XY2500V-C(5.08)-3P:XY2500V-C(5.08)-3P
- added JP2: GND_BRIGDE, Connector_PinSocket_2.54mm:PinSocket_2x03_P2.54mm_Vertical, symbol Connector_Generic:Conn_02x03_Odd_Even
- added L1, L2, L3, L4: LIM, XY2500V-C(5.08)-3P:XY2500V-C(5.08)-3P, symbol XY2500V-C(5.08)-3P:XY2500V-C(5.08)-3P
- added PON1: POWER_ON_SWITCHES, XY2500V-C(5.08)-4P:XY2500V-C(5.08)-4P, symbol XY2500V-C(5.08)-4P:XY2500V-C(5.08)-4P
- added R3: R, Resistor_SMD:R_0805_2012Metric, symbol Device:R
- added V1, V2, V3: V, XY2500V-C(5.08)-2P:XY2500V-C(5.08)-2P, symbol XY2500V-C(5.08)-2P:XY2500V-C(5.08)-2P
- added VA1, VA2, VA3: VA, XY2500V-C(5.08)-2P:XY2500V-C(5.08)-2P, symbol XY2500V-C(5.08)-2P:XY2500V-C(5.08)-2P
- E1: renamed from J45; footprint (none) -> MountingHole:MountingHole_4.5mm_Pad
- IN1: renamed from U12; value ~ -> IN1
- IN2: renamed from U17; value ~ -> IN2
- IN3: renamed from U18; value ~ -> IN3
- IN4: renamed from U13; value ~ -> IN4
- IN5: renamed from U14; value ~ -> IN5
- IN6: renamed from U15; value ~ -> IN6
- IN7: renamed from U16; value ~ -> IN7
- OUT1: renamed from U1; value ~ -> OUT1
- OUT2: renamed from U2; value ~ -> OUT2
- OUT3: renamed from U3; value ~ -> OUT3
- OUT34: renamed from U21; value ~ -> OUT34
- OUT4: renamed from U4; value ~ -> OUT4
- OUT5: renamed from U5; value ~ -> OUT5
- OUT6: renamed from U6; value ~ -> OUT6
- OUT7: renamed from U7; value ~ -> OUT7
- OUT8: renamed from U8; value ~ -> OUT8
- R1: renamed from R2; footprint Resistor_THT:R_Axial_DIN0207_L6.3mm_D2.5mm_P10.16mm_Horizontal -> Resistor_SMD:R_0805_2012Metric
- R2: renamed from R1; footprint Resistor_THT:R_Axial_DIN0207_L6.3mm_D2.5mm_P10.16mm_Horizontal -> Resistor_SMD:R_0805_2012Metric
- S1: renamed from U9; value ~ -> S1
- S2: renamed from U10; value ~ -> S2
- S3: renamed from U11; value ~ -> S3
- SS1: renamed from U19; value ~ -> SS1
- SS2: renamed from U20; value ~ -> SS2
- renumbered JJ1 to A1, D2 to D1, D1 to D2, J2 to DBI1, J1 to DBO1, J30 to JP1
Connections:
- net 200_NORMAL: now also J3.2
- net 202_24V: now also J2.1, R3.1, VA1.1, VA1.2, VA2.1, VA2.2, VA3.1, VA3.2
- net 204_24V/a: now also R2.1, J3.1; no longer R1.1
- net EXTERNAL_ESTOP: now also PON1.4
- net EXT_PWR: now also R1.1, J1.1; no longer R2.1
- net Earth: no longer A1.0 (PAD)
- net GND: now also RJ1.4, RJ1.5, SS2.3, SS2.4, G1.1, G1.2, G2.1, G2.2, G3.1, G3.2, J1.2, J3.3, JP2.1 (Pin_1), JP2.3 (Pin_3), JP2.5 (Pin_5), L1.1, L2.1, L3.1, L4.1
- net LIMIT_X: now also L1.2
- net LIMIT_Α: now also L4.2
- net LIMIT_Ζ: now also L3.2
- net LIMIT_Υ: now also L2.2
- net POWER_SWITCH: now also PON1.2
- net VDC: now also L1.3, L2.3, L3.3, L4.3, PON1.1, PON1.3, V1.1, V1.2, V2.1, V2.2, V3.1, V3.2
- net SS_5VP: now reaches SS1.1
- net SS_5VP: now also RJ1.7, RJ1.8, SS1.2; no longer RJ1.1
- net SS_TX+: now reaches RJ1.2
- net SS_TX+: now also SS2.1; no longer SS1.2
- net SS_RX+: now reaches SS1.3
- net SS_RX+: now also RJ1.6; no longer RJ1.3
- net SS_RX-: now reaches SS1.4
- net SS_RX-: now also RJ1.3; no longer RJ1.4
- net SS_TX-: now reaches SS2.2
- net SS_TX-: now also RJ1.1; no longer RJ1.6
- new net: D3.2 (A), R3.2
- new net GNDA: D3.1 (K), GA1.1, GA1.2, GA2.1, GA2.2, GA3.1, GA3.2, J2.2, JP2.2 (Pin_2), JP2.4 (Pin_4), JP2.6 (Pin_6)
- no-connect marks 62 -> 63
Other:
- note added: "IN0"
- note added: "IN1"
- note added: "IN10"
- note added: "IN11"
- note added: "IN12"
- note added: "IN2"
- note added: "IN3"
- note added: "IN4"
- note added: "IN5"
- note added: "IN6"
- note added: "IN7"
- note added: "IN8"
- note added: "IN9"
- moved on the sheet: A1, D1, D2, DBI1, DBO1, E1, H1, H2, H3, H4, H5, H6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

Commit message: board
Parts:
- removed J1: PWR, XY2500V-C(5.08)-2P:XY2500V-C(5.08)-2P, symbol XY2500V-C(5.08)-2P:XY2500V-C(5.08)-2P
- removed J2: V2, XY2500V-C(5.08)-2P:XY2500V-C(5.08)-2P, symbol XY2500V-C(5.08)-2P:XY2500V-C(5.08)-2P
- removed J3: V1, XY2500V-C(5.08)-3P:XY2500V-C(5.08)-3P, symbol XY2500V-C(5.08)-3P:XY2500V-C(5.08)-3P
- removed L1, L2, L3, L4: LIM, XY2500V-C(5.08)-3P:XY2500V-C(5.08)-3P, symbol XY2500V-C(5.08)-3P:XY2500V-C(5.08)-3P
- removed PON1: POWER_ON_SWITCHES, XY2500V-C(5.08)-4P:XY2500V-C(5.08)-4P, symbol XY2500V-C(5.08)-4P:XY2500V-C(5.08)-4P
- added G4, G5, IX4, IX5, IX6, IX7, IX8, IX9, U1, U3, V4, V5: XY2500R-C(5.08)-2P, XY2500R-C(5.08)-2P:XY2500R-C(5.08)-2P, symbol XY2500R-C(5.08)-2P:XY2500R-C(5.08)-2P
- added IN8: IN, XY2500V-C(5.08)-3P:XY2500V-C(5.08)-3P, symbol XY2500V-C(5.08)-3P:XY2500V-C(5.08)-3P
- added IX1, IX2, IX3, U2: XY2500R-C(5.08)-3P, XY2500R-C(5.08)-3P:XY2500R-C(5.08)-3P, symbol XY2500R-C(5.08)-3P:XY2500R-C(5.08)-3P
- IN1: value IN1 -> IN
- IN2: value IN2 -> IN
- IN3: value IN3 -> IN
- IN4: value IN4 -> IN
- IN5: value IN5 -> IN
- IN6: value IN6 -> IN
- IN7: value IN7 -> IN
- OUT1: value OUT1 -> OUT
- OUT2: value OUT2 -> OUT
- OUT3: value OUT3 -> OUT
- OUT34: value OUT34 -> OUT
- OUT4: value OUT4 -> OUT
- OUT5: value OUT5 -> OUT
- OUT6: value OUT6 -> OUT
- OUT7: value OUT7 -> OUT
- OUT8: value OUT8 -> OUT
Connections:
- net EXTERNAL_ESTOP is gone; now on net LIMIT_X: IN1.1
- net LIMIT_Α is gone; now on net 19X7_HANDWHEEL_Z: IN3.2
- net POWER_SWITCH is gone; now on net LIMIT_Υ: IN1.2
- net 19X7_24V: now also IN4.1; no longer IN5.2
- net 19X7_HANDWHEEL_X: now also IN2.2; no longer IN4.1
- net 19X7_HANDWHEEL_Y: now also DBI1.3, IN3.1; no longer DBI1.2, IN4.2
- net 19X7_HANDWHEEL_Z: now also DBI1.2; no longer DBI1.3, IN5.1
- net 19X7_LUBRICANT: now also IN5.2; no longer IN7.1
- net 19X7_MAIN_DRIVE_OFF: now also IN4.2; no longer IN6.1
- net 19X7_NOT_SPINDLE_FEED: now also IN5.1; no longer IN6.2
- net 200_NORMAL: now also U2.2
- net 202_24V: now also U3.1
- net 204_24V/a: now also U2.1
- net EXT_PWR: now also U1.1
- net Earth: now also A1.0 (PAD)
- net GND: now also SS1.1, SS1.2, G4.1, G4.2, G5.1, G5.2, IN8.3, IX1.1, IX2.1, IX3.1, U1.2, U2.3; no longer SS2.3, SS2.4
- net GNDA: now also U3.2
- net LIMIT_X: now also IX1.2; no longer IN2.1
- net LIMIT_Ζ: now also IN2.1, IX3.2; no longer IN3.1
- net LIMIT_Υ: now also IX2.2; no longer IN2.2
- net SS_5VP: now also SS2.3, SS2.4; no longer SS1.1, SS1.2
- net VDC: now also IX1.3, IX2.3, IX3.3, IX4.2, IX5.2, IX6.2, IX7.2, IX8.2, IX9.2, V4.1, V4.2, V5.1, V5.2
- net IN13: now reaches IN7.2
- net IN13: now also IX7.1
- new net IN10: IN6.1, IX4.1
- new net IN11: IN6.2, IX5.1
- new net IN12: IN7.1, IX6.1
- new net IN14: IN8.1, IX8.1
- new net IN15: IN8.2, IX9.1
- no-connect marks 63 -> 61
Other:
- note added: "IN13"
- note added: "IN14"
- note added: "IN15"
- moved on the sheet: A1, D1, D2, D3, DBI1, DBO1, E1, G1, G2, G3, GA1, GA2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

Commit message: maho-io release for fab
Parts:
- removed OUT1, OUT2, OUT3: OUT, XY2500V-C(5.08)-2P:XY2500V-C(5.08)-2P, symbol XY2500V-C(5.08)-2P:XY2500V-C(5.08)-2P
- added OUTX1, OUTX2, OUTX3: XY2500R-C(5.08)-2P, XY2500R-C(5.08)-2P:XY2500R-C(5.08)-2P, symbol XY2500R-C(5.08)-2P:XY2500R-C(5.08)-2P
- renumbered OUT34 to OUT1, OUT4 to OUT2, OUT5 to OUT3, OUT6 to OUT4, OUT7 to OUT5, OUT8 to OUT6
Connections:
- net 19X6_HANDWHEEL_X: now also OUTX1.1
- net 19X6_HANDWHEEL_Y: now also OUTX2.1
- net 19X6_HANDWHEEL_Z: now also OUTX3.1
- net 200_NORMAL: now also OUTX1.2, OUTX2.2, OUTX3.2
- net 19X7_24V renamed 19X7_200_HIGH
- net IN10 renamed EXT_ESTOP
- net IN11 renamed PON_SWITCH
Other:
- moved on the sheet: DBI1, IN1, IN2, IN3, IN4, IN5, IN6, IN7, IN8, IX1, IX2, IX3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

Commit message: updates analog
Other:
- note added: "ANALOG_X1"
- note added: "ANALOG_X2"
- note added: "ANALOG_Y1"
- note added: "ANALOG_Y2"
- note added: "ANALOG_Z1"
- note added: "ANALOG_Z2"
- moved on the sheet: A1, S1, S2, S3
