File: retrofit/master/master.kicad_sch (KiCad schematic)
At the start: 22 parts, among them J1 PWR, J2 MAHO CTRL, J3 Proximity X, J4 Proximity X, J5 Proximity X, U10 7i97-TB5-Inputs-D, U11 7i97-TB4-Inputs-A, U2 7i97-TB4-RS485, U3 7i97-TB3-ANALOG-A, U5 7i97-TB3-ANALOG-B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

Commit message: updates
Parts:
- added U18: 7i97-ENC2, symbol MAHO:7i97-ENC2
Other:
- note added: "Add 7i84 Wiring"
- note added: "Add here spindle speed encoder"
- moved on the sheet: B?, J1, J2, J3, J4, J5, J?, U10, U11, U2, U3, U5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

Commit message: updates
Parts:
- removed U18: 7i97-ENC2, symbol MAHO:7i97-ENC2
- added U18: 7i97-ENC5, symbol MAHO:7i97-ENC5
Changed lines of the file:
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@@
 	(text "Add 7i84 Wiring	"
 		(exclude_from_sim no)
-		(at 294.64 133.35 0)
+		(at 279.146 73.66 0)
 		(effects
 			(font
@@
 	(text "Add here spindle speed encoder"
 		(exclude_from_sim no)
-		(at 93.98 246.38 0)
+		(at 67.31 245.618 0)
 		(effects
 			(font
@@
 	)
 	(symbol
-		(lib_id "MAHO:7i97-ENC2")
-		(at 189.23 245.11 0)
-		(unit 1)
-		(exclude_from_sim no)
-		(in_bom yes)
-		(on_board yes)
-		(dnp no)
-		(property "Reference" "U18"
-			(at 187.96 228.6 0)
-			(effects
-				(font
-					(size 1.27 1.27)
-				)
-				(justify left)
-			)
-		)
-		(property "Value" "7i97-ENC2"
-			(at 184.15 231.14 0)
-			(effects
-				(font
-					(size 1.27 1.27)
-				)
-				(justify left)
-			)
-		)
-		(property "Footprint" ""
-			(at 245.745 158.75 0)
-			(effects
-				(font
-					(size 1.27 1.27)
-				)
-				(hide yes)
-			)
-		)
-		(property "Datasheet" ""
-			(at 245.745 158.75 0)
-			(effects
-				(font
-					(size 1.27 1.27)
-				)
-				(hide yes)
-			)
-		)
-		(property "Description" ""
-			(at 189.23 245.11 0)
-			(effects
-				(font
-					(size 1.27 1.27)
-				)
-				(hide yes)
-			)
-		)
-		(pin "17"
-		)
-		(pin "18"
-		)
-		(pin "19"
-		)
-		(pin "20"
-		)
-		(pin "21"
-		)
-		(pin "22"
-		)
-		(pin "23"
-		)
-		(pin "24"
-		)
-		(instances
-			(project "master"
-				(path "/6b7450d6-3952-419a-ab30-dcf88fa68fd4"
-					(reference "U18")
-					(unit 1)
-				)
-			)
-		)
-	)
-	(symbol
 		(lib_id "MAHO:Breakout")
 		(at 102.87 83.82 0)
@@
 					(unit 1)
 				)
+			)
+		)
+	)
+	(symbol
+		(lib_id "MAHO:7i97-ENC5")
+		(at 199.39 250.19 0)
+		(unit 1)
+		(exclude_from_sim no)
+		(in_bom yes)
+		(on_board yes)
+		(dnp no)
+		(fields_autoplaced yes)
+		(property "Reference" "U18"
+			(at 204.47 248.9199 0)
+			(effects
+				(font
+					(size 1.27 1.27)
+				)
+				(justify left)
+			)
+		)
+		(property "Value" "7i97-ENC5"
+			(at 204.47 251.4599 0)
+			(effects
+				(font
+					(size 1.27 1.27)
+				)
+				(justify left)
+			)
+		)
+		(property "Footprint" ""
+			(at 255.905 163.83 0)
+			(effects
+				(font
+					(size 1.27 1.27)
+				)
+				(hide yes)
+			)
+		)
+		(property "Datasheet" ""
+			(at 255.905 163.83 0)
+			(effects
+				(font
+					(size 1.27 1.27)
+				)
+				(hide yes)
+			)
+		)
+		(property "Description" ""
+			(at 199.39 250.19 0)
+			(effects
+				(font
+					(size 1.27 1.27)
+				)
+				(hide yes)
+			)
+		)
+		(pin "20"
+		)
+		(pin "19"
+		)
+		(pin "21"
+		)
+		(pin "23"
+		)
+		(pin "24"
+		)
+		(pin "18"
+		)
+		(pin "17"
+		)
+		(pin "22"
+		)
+		(instances
+			(project ""
+				(path "/6b7450d6-3952-419a-ab30-dcf88fa68fd4"
+					(reference "U18")
+					(unit 1)
+				)
