File: retrofit/master/LinearEncoders.kicad_sch (KiCad schematic)
At the start: 9 parts, among them U1 7i97-ENC0, U4 7i97-ENC1, U7 7i97-ENC2

Commit message: updates
Connections:
- net at EXE?.2 ((Yellow)_Ie1B): now also LS?.2 ((Yellow)_Ie1B) (x3)
- net at EXE?.7 ((Violet)_/Uas): now also LS?.7 ((Gray)_Ie0A) (x3)
- net at EXE?.8 (SHIELD): now also U1.4 (QB0); no longer LS?.8 (SHIELD)
- new net: EXE?.8 (SHIELD), LS?.8 (SHIELD) (x3)
Changed lines of the file:
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@@
     (pin "24")
     (instances
-      (project "retrofit"
+      (project "master"
         (path "/6b7450d6-3952-419a-ab30-dcf88fa68fd4"
           (reference "U7") (unit 1)
@@
     (pin "9")
     (instances
-      (project "retrofit"
+      (project "master"
         (path "/6b7450d6-3952-419a-ab30-dcf88fa68fd4"
           (reference "EXE?") (unit 1)
@@
     (pin "9")
     (instances
-      (project "retrofit"
+      (project "master"
         (path "/6b7450d6-3952-419a-ab30-dcf88fa68fd4"
           (reference "EXE?") (unit 1)
@@
     (pin "9")
     (instances
-      (project "retrofit"
+      (project "master"
         (path "/6b7450d6-3952-419a-ab30-dcf88fa68fd4"
           (reference "U4") (unit 1)
@@
     (pin "9")
     (instances
-      (project "retrofit"
+      (project "master"
         (path "/6b7450d6-3952-419a-ab30-dcf88fa68fd4"
           (reference "EXE?") (unit 1)
@@
     (pin "8")
     (instances
-      (project "retrofit"
+      (project "master"
         (path "/6b7450d6-3952-419a-ab30-dcf88fa68fd4"
           (reference "LS?") (unit 1)
@@
     (pin "8")
     (instances
-      (project "retrofit"
+      (project "master"
         (path "/6b7450d6-3952-419a-ab30-dcf88fa68fd4"
           (reference "LS?") (unit 1)
@@
     (pin "8")
     (instances
-      (project "retrofit"
+      (project "master"
         (path "/6b7450d6-3952-419a-ab30-dcf88fa68fd4"
           (reference "LS?") (unit 1)
@@
     (pin "8")
     (instances
-      (project "retrofit"
+      (project "master"
         (path "/6b7450d6-3952-419a-ab30-dcf88fa68fd4"
           (reference "U1") (unit 1)

Commit message: cleanup
Parts:
- gave numbers to parts that had none: 6
- renumbered U4 to U12, U7 to U15
Connections:
- net at U14.2 ((Yellow)_Ie1B): now also U13.2 ((Yellow)_Ie1B)
- net at U14.7 ((Violet)_/Uas): now also U13.7 ((Gray)_Ie0A)
- net at U17.2 ((Yellow)_Ie1B): now also U16.2 ((Yellow)_Ie1B)
- net at U17.7 ((Violet)_/Uas): now also U16.7 ((Gray)_Ie0A)
- net at U7.2 ((Yellow)_Ie1B): now also U4.2 ((Yellow)_Ie1B)
- net at U7.7 ((Violet)_/Uas): now also U4.7 ((Gray)_Ie0A)
- net at U7.8 (SHIELD): now also U1.4 (QB0); no longer U4.8 (SHIELD)
- new net: U13.8 (SHIELD), U14.8 (SHIELD)
- new net: U16.8 (SHIELD), U17.8 (SHIELD)
- new net: U4.8 (SHIELD), U7.8 (SHIELD)

Commit message: updates
Connections:
- net at U14.2 ((Blue)_/5V_Sensor): now also U13.2 ((Yellow)_Ie1B)
- net at U14.7 ((Violet)_/Uas): now also U13.7 ((Gray)_Ie0A)
- net at U17.2 ((Blue)_/5V_Sensor): now also U16.2 ((Yellow)_Ie1B)
- net at U17.7 ((Violet)_/Uas): now also U16.7 ((Gray)_Ie0A)
- net at U7.2 ((Blue)_/5V_Sensor): now also U4.2 ((Yellow)_Ie1B)
- net at U7.7 ((Violet)_/Uas): now also U4.7 ((Gray)_Ie0A)
- net at U7.8 ((Gray)_Ua2): now also U1.4 (QB0); no longer U4.8 (SHIELD)
- new net: U13.8 (SHIELD), U14.8 ((Gray)_Ua2)
- new net: U16.8 (SHIELD), U17.8 ((Gray)_Ua2)
- new net: U4.8 (SHIELD), U7.8 ((Gray)_Ua2)

Commit message: updates
Connections:
- net at U14.2 ((Blue)_/5V_Sensor): now also U13.2 ((Yellow)_Ie1B)
- net at U14.7 ((Violet)_/Uas): now also U13.7 ((Gray)_Ie0A)
- net at U17.2 ((Blue)_/5V_Sensor): now also U16.2 ((Yellow)_Ie1B)
- net at U17.7 ((Violet)_/Uas): now also U16.7 ((Gray)_Ie0A)
- net at U7.2 ((Blue)_/5V_Sensor): now also U4.2 ((Yellow)_Ie1B)
- net at U7.7 ((Violet)_/Uas): now also U4.7 ((Gray)_Ie0A)
- net at U7.8 ((Gray)_Ua2): now also U1.4 (QB0); no longer U4.8 (SHIELD)
- new net: U13.8 (SHIELD), U14.8 ((Gray)_Ua2)
- new net: U16.8 (SHIELD), U17.8 ((Gray)_Ua2)
- new net: U4.8 (SHIELD), U7.8 ((Gray)_Ua2)
Changed lines of the file:
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@@
 					(at -8.89 3.81 0)
 					(length 5.08)
-					(name "GB2"
+					(name "QB2"
 						(effects
 							(font
@@
 					(at -8.89 1.27 0)
 					(length 5.08)
-					(name "/GB2"
+					(name "/QB2"
 						(effects
 							(font

Commit message: updates
Connections:
- net at U14.2 ((Blue)_/5V_Sensor): now also U13.2 ((Yellow)_Ie1B)
- net at U14.7 ((Violet)_/Uas): now also U13.7 ((Gray)_Ie0A)
- net at U17.2 ((Blue)_/5V_Sensor): now also U16.2 ((Yellow)_Ie1B)
- net at U17.7 ((Violet)_/Uas): now also U16.7 ((Gray)_Ie0A)
- net at U7.2 ((Blue)_/5V_Sensor): now also U4.2 ((Yellow)_Ie1B)
- net at U7.7 ((Violet)_/Uas): now also U4.7 ((Gray)_Ie0A)
- net at U7.8 ((Gray)_Ua2): now also U1.4 (QB0); no longer U4.8 (SHIELD)
- new net: U13.8 (SHIELD), U14.8 ((Gray)_Ua2)
- new net: U16.8 (SHIELD), U17.8 ((Gray)_Ua2)
- new net: U4.8 (SHIELD), U7.8 ((Gray)_Ua2)
